File: NES_EMULATOR.kicad_pcb (KiCad board)
At the start: 2 copper layers, 123.4 x 123 mm, 34 parts, among them SW1 SW_MEC_5E, SW2 SW_MEC_5E, SW3 SW_MEC_5E, SW4 SW_MEC_5E, SW5 SW_MEC_5E, SW6 SW_MEC_5E, SW7 SW_MEC_5E, SW8 SW_MEC_5E, U1 NES_LCD, U2 FK723M1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

Commit message: Fixed pcb design
Parts:
- C10, C11, C3, C4, C6, C7, C9: moved to F.Cu
- U4: footprint Package_SO:SSOP-8_2.95x2.8mm_P0.65mm -> Package_SO:SOIC-8_3.9x4.9mm_P1.27mm
- moved C2 55.5 mm to (61.4, 71.5), turned to 0 degrees
- moved C3 43.2 mm to (114.8, 59.9), turned to 90 degrees
- moved C10 13.6 mm to (27.4, 96.8)
- moved C11 12.5 mm to (34.2, 85.3), turned to -90 degrees
- moved C7 12.1 mm to (21.5, 95.7), turned to 90 degrees
- moved C4 7.60 mm to (59.7, 108.8)
- moved C6 7.49 mm to (63.8, 108.8)
- moved C9 3.10 mm to (20.8, 99.0)
- moved C13 0.97 mm to (91.2, 83.5)
- moved U4 0.71 mm to (85.6, 82.8)
- moved LS1 0.20 mm to (61.7, 89.7)
Connections:
- U1 pad 35: (no net) -> unconnected-(U1-MH-Pad35)
- U1 pad 36: (no net) -> unconnected-(U1-MH-Pad36)
Routing:
- net RIGHT_BTN: track 218.1 -> 222.6 mm
- net LEFT_BTN: track 68.9 -> 72.3 mm
- net DOWN_BTN: track 132.9 -> 129.8 mm
- net B_BTN: track 130.8 -> 133.6 mm
- net AUDIO_SHTDN: track 27.8 -> 25.4 mm
- net ~{LCD_RST}: track 108.3 -> 106.6 mm
- net UP_BTN: track 73.2 -> 71.7 mm
- net GND: track 3.38 -> 2.09 mm, vias 17 -> 43
- net A_BTN: track 92.0 -> 91.0 mm
- net Net-(U4-+IN): track 6.52 -> 7.38 mm
- net LCD_BL: track 26.1 -> 25.4 mm
- net Net-(U4-VO2): track 40.3 -> 39.7 mm
- net SELECT_BTN: track 220.4 -> 220.8 mm, vias 5 -> 4
