File: NES_EMULATOR.kicad_sch (KiCad schematic)
At the start: 34 parts, among them SW1 SW_MEC_5E, SW2 SW_MEC_5E, SW3 SW_MEC_5E, SW4 SW_MEC_5E, SW5 SW_MEC_5E, SW6 SW_MEC_5E, SW7 SW_MEC_5E, SW8 SW_MEC_5E, U1 NES_LCD, U2 FK723M1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

Commit message: Fixed pcb design
Parts:
- U4: footprint Package_SO:SSOP-8_2.95x2.8mm_P0.65mm -> Package_SO:SOIC-8_3.9x4.9mm_P1.27mm
Connections:
- no-connect marks 84 -> 86
